Commit message: update files

File: urdf/mycobot_280_m5.urdf.xacro (robot description, xacro)
@@ -14,6 +14,5 @@
       <geometry>
 	     <!--- 0.0 0 -0.04  1.5708 3.14159-->
-       <!-- <mesh filename="file:///($find gazebo_simulation_ros2)/urdf/joint1.dae"/> -->
-       <mesh filename="package://gazebo_simulation_ros2/urdf/joint1.dae"/>
+       <mesh filename="file://$(find gazebo_simulation_ros2)/urdf/joint1.dae"/>
       </geometry>
       <origin xyz = "0.0 0 0 " rpy = " 0 0 -1.5708"/>
@@ -22,5 +21,5 @@
       <geometry>
 	     <!--- 0.0 0 -0.04  1.5708 3.14159-->
-       <mesh filename="file:///($find gazebo_simulation_ros2)/urdf/joint1.dae"/>
+       <mesh filename="file://$(find gazebo_simulation_ros2)/urdf/joint1.dae"/>
         </geometry>
         <origin xyz = "0.0 0 0.0 " rpy = " 0 0 -1.5708"/>
@@ -38,5 +37,5 @@
     <visual>
       <geometry>
-       <mesh filename="file:///($find gazebo_simulation_ros2)/urdf/joint2.dae"/>
+       <mesh filename="file://$(find gazebo_simulation_ros2)/urdf/joint2.dae"/>
       </geometry>
       <origin xyz = "0.0 0 -0.061 " rpy = " 0 0 -1.5708"/>
@@ -44,5 +43,5 @@
     <collision>
      <geometry>
-       <mesh filename="file:///($find gazebo_simulation_ros2)/urdf/joint2.dae"/>
+       <mesh filename="file://$(find gazebo_simulation_ros2)/urdf/joint2.dae"/>
       </geometry>
       <origin xyz = "0.0 0 -0.061 " rpy = " 0 0 -1.5708"/>
@@ -60,5 +59,5 @@
     <visual>
       <geometry>
-       <mesh filename="file:///($find gazebo_simulation_ros2)/urdf/joint3.dae"/>
+       <mesh filename="file://$(find gazebo_simulation_ros2)/urdf/joint3.dae"/>
       </geometry>
     <origin xyz = "0.0 0 0.03256 " rpy = " 0 -1.5708 0"/>
@@ -66,5 +65,5 @@
     <collision>
       <geometry>
-       <mesh filename="file:///($find gazebo_simulation_ros2)/urdf/joint3.dae"/>
+       <mesh filename="file://$(find gazebo_simulation_ros2)/urdf/joint3.dae"/>
       </geometry>
       <origin xyz = "0.00 0 0.03256 " rpy = " 0 -1.5708 0"/>
@@ -83,5 +82,5 @@
       <geometry>
        <!--- 0.0 0 -0.04 -->
-       <mesh filename="file:///($find gazebo_simulation_ros2)/urdf/joint4.dae"/>
+       <mesh filename="file://$(find gazebo_simulation_ros2)/urdf/joint4.dae"/>
       </geometry>
       <origin xyz = "0.0 0 0.03056 " rpy = " 0 -1.5708 0"/>
@@ -90,5 +89,5 @@
       <geometry>
        <!--- 0.0 0 -0.04 -->
-       <mesh filename="file:///($find gazebo_simulation_ros2)/urdf/joint4.dae"/>
+       <mesh filename="file://$(find gazebo_simulation_ros2)/urdf/joint4.dae"/>
       </geometry>
       <origin xyz = "-0.0 0 0.03056 " rpy = " 0 -1.5708 0"/>
@@ -107,5 +106,5 @@
       <geometry>
        <!--- 0.0 0 -0.04 -->
-       <mesh filename="file:///($find gazebo_simulation_ros2)/urdf/joint5.dae"/>
+       <mesh filename="file://$(find gazebo_simulation_ros2)/urdf/joint5.dae"/>
       </geometry>
       <origin xyz = "0.0 0 -0.0340 " rpy = " -1.5708 0 0"/>
@@ -114,5 +113,5 @@
        <geometry>
        <!--- 0.0 0 -0.04 -->
-       <mesh filename="file:///($find gazebo_simulation_ros2)/urdf/joint5.dae"/>
+       <mesh filename="file://$(find gazebo_simulation_ros2)/urdf/joint5.dae"/>
       </geometry>
       <origin xyz = "0.0 0 -0.0340 " rpy = " -1.5708 0 0"/>
@@ -131,5 +130,5 @@
       <geometry>
        <!--- 0.0 0 -0.04 -->
-       <mesh filename="file:///($find gazebo_simulation_ros2)/urdf/joint6.dae"/>
+       <mesh filename="file://$(find gazebo_simulation_ros2)/urdf/joint6.dae"/>
       </geometry>
     <origin xyz = "-0.00 0.0 -0.044 " rpy = " 0 0 0"/>
@@ -138,5 +137,5 @@
       <geometry>
        <!--- 0.0 0 -0.04 -->
-       <mesh filename="file:///($find gazebo_simulation_ros2)/urdf/joint6.dae"/>
+       <mesh filename="file://$(find gazebo_simulation_ros2)/urdf/joint6.dae"/>
       </geometry>
     <origin xyz = "-0.00 0.0 -0.044 " rpy = " 0 0 0"/>
@@ -155,6 +154,6 @@
       <geometry>
        <!--- 0.0 0 -0.04 -->
-       <box size="1 1 1"/>
-       <!-- <mesh filename="file:///($find gazebo_simulation_ros2)/urdf/joint7.dae"/> -->
+       <!-- <box size="1 1 1"/> -->
+       <mesh filename="file://$(find gazebo_simulation_ros2)/urdf/joint7.dae"/>
       </geometry>
     <origin xyz = "-0.00 0.00 -0.014 " rpy = " 0 0 0"/>
@@ -163,5 +162,5 @@
       <geometry>
        <!--- 0.0 0 -0.04 -->
-       <mesh filename="file:///($find gazebo_simulation_ros2)/urdf/joint7.dae"/>
+       <mesh filename="file://$(find gazebo_simulation_ros2)/urdf/joint7.dae"/>
       </geometry>
     <origin xyz = "-0.00 0.00 -0.014 " rpy = " 0 0 0"/>
@@ -216,11 +215,12 @@
 </joint>
     <!-- for gazebo simulation -->
-    <!-- <gazebo>
-      <plugin name="gazebo_ros_control" filename="libgazebo_ros_control.so">
-        <robotNamespace>/myCobot</robotNamespace>
-        <robotSimType>gazebo_ros_control/DefaultRobotHWSim</robotSimType>
-        <legacyModeNS>false</legacyModeNS>
-      </plugin>
-    </gazebo> -->
+    <gazebo>
+      <plugin filename="libgazebo_ros2_control.so" name="gazebo_ros2_control">
+        <!-- <robot_param>robot_description</robot_param>
+        <robot_param_node>robot_state_publisher</robot_param_node> -->
+        <parameters>$(find gazebo_simulation_ros2)/config/fake_ros2_control.yaml</parameters>
+      <!-- <parameters>$(find manta_v2_gazebo_ros2_control)/config/manta_v2_trajectory_controller.yaml</parameters> -->
+    </plugin>
+  </gazebo>
 <!-- ros2_control -->
 <ros2_control name="GazeboSystem" type="system">
@@ -228,72 +228,64 @@
     <plugin>gazebo_ros2_control/GazeboSystem</plugin>
     </hardware>
+      <transmission name="joint1_trans">
+        <type>transmission_interface/SimpleTransmission</type>
+        <joint name="joint1">
+          <hardwareInterface>hardware_interface/PositionJointInterface</hardwareInterface>
+        </joint>
+        <actuator name="joint1_motor">
+          <hardwareInterface>hardware_interface/PositionJointInterface</hardwareInterface>
+          <mechanicalReduction>1</mechanicalReduction>
+        </actuator>
+      </transmission>
+      <transmission name="joint2_trans">
+        <type>transmission_interface/SimpleTransmission</type>
+        <joint name="joint2">
+          <hardwareInterface>hardware_interface/PositionJointInterface</hardwareInterface>
+        </joint>
+        <actuator name="joint2_motor">
+          <hardwareInterface>hardware_interface/PositionJointInterface</hardwareInterface>
+          <mechanicalReduction>1</mechanicalReduction>
+        </actuator>
+      </transmission>
+      <transmission name="joint3_trans">
+        <type>transmission_interface/SimpleTransmission</type>
+        <joint name="joint3">
+          <hardwareInterface>hardware_interface/PositionJointInterface</hardwareInterface>
+        </joint>
+        <actuator name="joint3_motor">
+          <hardwareInterface>hardware_interface/PositionJointInterface</hardwareInterface>
+          <mechanicalReduction>1</mechanicalReduction>
+        </actuator>
+      </transmission>
+      <transmission name="joint4_trans">
+        <type>transmission_interface/SimpleTransmission</type>
+        <joint name="joint4">
+          <hardwareInterface>hardware_interface/PositionJointInterface</hardwareInterface>
+        </joint>
+        <actuator name="joint4_motor">
+          <hardwareInterface>hardware_interface/PositionJointInterface</hardwareInterface>
+          <mechanicalReduction>1</mechanicalReduction>
+        </actuator>
+      </transmission>
+      <transmission name="joint5_trans">
+        <type>transmission_interface/SimpleTransmission</type>
+        <joint name="joint5">
+          <hardwareInterface>hardware_interface/PositionJointInterface</hardwareInterface>
+        </joint>
+        <actuator name="joint5_motor">
+          <hardwareInterface>hardware_interface/PositionJointInterface</hardwareInterface>
+          <mechanicalReduction>1</mechanicalReduction>
+        </actuator>
+      </transmission>
+      <transmission name="joint6_trans">
+        <type>transmission_interface/SimpleTransmission</type>
+        <joint name="joint6">
+          <hardwareInterface>hardware_interface/PositionJointInterface</hardwareInterface>
+        </joint>
+        <actuator name="joint6_motor">
+          <hardwareInterface>hardware_interface/PositionJointInterface</hardwareInterface>
+          <mechanicalReduction>1</mechanicalReduction>
+        </actuator>
+      </transmission>
 </ros2_control>
-<!-- <gazebo>
-  <plugin filename="libgazebo_ros2_control.so" name="gazebo_ros2_control">
-    <robot_param>robot_description</robot_param>
-    <robot_param_node>robot_state_publisher</robot_param_node>
-    <parameters>$(find gazebo_simulation_ros2)/config/fake_ros2_control.yaml</parameters>
-      <parameters>$(find manta_v2_gazebo_ros2_control)/config/manta_v2_trajectory_controller.yaml</parameters>
-    </plugin>
-  </gazebo> -->
-      <transmission name="joint1_trans">
-        <type>transmission_interface/SimpleTransmission</type>
-        <joint name="joint1">
-          <hardwareInterface>hardware_interface/PositionJointInterface</hardwareInterface>
-        </joint>
-        <actuator name="joint1_motor">
-          <hardwareInterface>hardware_interface/PositionJointInterface</hardwareInterface>
-          <mechanicalReduction>1</mechanicalReduction>
-        </actuator>
-      </transmission>
-      <transmission name="joint2_trans">
-        <type>transmission_interface/SimpleTransmission</type>
-        <joint name="joint2">
-          <hardwareInterface>hardware_interface/PositionJointInterface</hardwareInterface>
-        </joint>
-        <actuator name="joint2_motor">
-          <hardwareInterface>hardware_interface/PositionJointInterface</hardwareInterface>
-          <mechanicalReduction>1</mechanicalReduction>
-        </actuator>
-      </transmission>
-      <transmission name="joint3_trans">
-        <type>transmission_interface/SimpleTransmission</type>
-        <joint name="joint3">
-          <hardwareInterface>hardware_interface/PositionJointInterface</hardwareInterface>
-        </joint>
-        <actuator name="joint3_motor">
-          <hardwareInterface>hardware_interface/PositionJointInterface</hardwareInterface>
-          <mechanicalReduction>1</mechanicalReduction>
-        </actuator>
-      </transmission>
-      <transmission name="joint4_trans">
-        <type>transmission_interface/SimpleTransmission</type>
-        <joint name="joint4">
-          <hardwareInterface>hardware_interface/PositionJointInterface</hardwareInterface>
-        </joint>
-        <actuator name="joint4_motor">
-          <hardwareInterface>hardware_interface/PositionJointInterface</hardwareInterface>
-          <mechanicalReduction>1</mechanicalReduction>
-        </actuator>
-      </transmission>
-      <transmission name="joint5_trans">
-        <type>transmission_interface/SimpleTransmission</type>
-        <joint name="joint5">
-          <hardwareInterface>hardware_interface/PositionJointInterface</hardwareInterface>
-        </joint>
-        <actuator name="joint5_motor">
-          <hardwareInterface>hardware_interface/PositionJointInterface</hardwareInterface>
-          <mechanicalReduction>1</mechanicalReduction>
-        </actuator>
-      </transmission>
-      <transmission name="joint6_trans">
-        <type>transmission_interface/SimpleTransmission</type>
-        <joint name="joint6">
-          <hardwareInterface>hardware_interface/PositionJointInterface</hardwareInterface>
-        </joint>
-        <actuator name="joint6_motor">
-          <hardwareInterface>hardware_interface/PositionJointInterface</hardwareInterface>
-          <mechanicalReduction>1</mechanicalReduction>
-        </actuator>
-      </transmission>
 </robot>

Commit message: update files

File: urdf/mycobot_280_m5.urdf.xacro (robot description, xacro)
@@ -214,78 +214,3 @@
   <child link="link1"/>
 </joint>
-    <!-- for gazebo simulation -->
-    <gazebo>
-      <plugin filename="libgazebo_ros2_control.so" name="gazebo_ros2_control">
-        <!-- <robot_param>robot_description</robot_param>
-        <robot_param_node>robot_state_publisher</robot_param_node> -->
-        <parameters>$(find gazebo_simulation_ros2)/config/fake_ros2_control.yaml</parameters>
-      <!-- <parameters>$(find manta_v2_gazebo_ros2_control)/config/manta_v2_trajectory_controller.yaml</parameters> -->
-    </plugin>
-  </gazebo>
-<!-- ros2_control -->
-<ros2_control name="GazeboSystem" type="system">
-  <hardware>
-    <plugin>gazebo_ros2_control/GazeboSystem</plugin>
-    </hardware>
-      <transmission name="joint1_trans">
-        <type>transmission_interface/SimpleTransmission</type>
-        <joint name="joint1">
-          <hardwareInterface>hardware_interface/PositionJointInterface</hardwareInterface>
-        </joint>
-        <actuator name="joint1_motor">
-          <hardwareInterface>hardware_interface/PositionJointInterface</hardwareInterface>
-          <mechanicalReduction>1</mechanicalReduction>
-        </actuator>
-      </transmission>
-      <transmission name="joint2_trans">
-        <type>transmission_interface/SimpleTransmission</type>
-        <joint name="joint2">
-          <hardwareInterface>hardware_interface/PositionJointInterface</hardwareInterface>
-        </joint>
-        <actuator name="joint2_motor">
-          <hardwareInterface>hardware_interface/PositionJointInterface</hardwareInterface>
-          <mechanicalReduction>1</mechanicalReduction>
-        </actuator>
-      </transmission>
-      <transmission name="joint3_trans">
-        <type>transmission_interface/SimpleTransmission</type>
-        <joint name="joint3">
-          <hardwareInterface>hardware_interface/PositionJointInterface</hardwareInterface>
-        </joint>
-        <actuator name="joint3_motor">
-          <hardwareInterface>hardware_interface/PositionJointInterface</hardwareInterface>
-          <mechanicalReduction>1</mechanicalReduction>
-        </actuator>
-      </transmission>
-      <transmission name="joint4_trans">
-        <type>transmission_interface/SimpleTransmission</type>
-        <joint name="joint4">
-          <hardwareInterface>hardware_interface/PositionJointInterface</hardwareInterface>
-        </joint>
-        <actuator name="joint4_motor">
-          <hardwareInterface>hardware_interface/PositionJointInterface</hardwareInterface>
-          <mechanicalReduction>1</mechanicalReduction>
-        </actuator>
-      </transmission>
-      <transmission name="joint5_trans">
-        <type>transmission_interface/SimpleTransmission</type>
-        <joint name="joint5">
-          <hardwareInterface>hardware_interface/PositionJointInterface</hardwareInterface>
-        </joint>
-        <actuator name="joint5_motor">
-          <hardwareInterface>hardware_interface/PositionJointInterface</hardwareInterface>
-          <mechanicalReduction>1</mechanicalReduction>
-        </actuator>
-      </transmission>
-      <transmission name="joint6_trans">
-        <type>transmission_interface/SimpleTransmission</type>
-        <joint name="joint6">
-          <hardwareInterface>hardware_interface/PositionJointInterface</hardwareInterface>
-        </joint>
-        <actuator name="joint6_motor">
-          <hardwareInterface>hardware_interface/PositionJointInterface</hardwareInterface>
-          <mechanicalReduction>1</mechanicalReduction>
-        </actuator>
-      </transmission>
-</ros2_control>
 </robot>

Commit message: update robot model files

File: urdf/mycobot_280_m5.urdf.xacro (robot description, xacro)
@@ -214,18 +214,79 @@
   <child link="link1"/>
 </joint>
-   <!-- for gazebo simulation -->
+  <ros2_control name="GazeboSystem" type="system">
+    <hardware>
+      <plugin>gazebo_ros2_control/GazeboSystem</plugin>
+    </hardware>
+    <joint name="joint1">
+      <command_interface name="position">
+        <param name="min">-3.15</param>
+        <param name="max">3.14</param>
+      </command_interface>
+      <state_interface name="position">
+        <param name="initial_value">0.0</param>
+      </state_interface>
+      <state_interface name="velocity"/>
+      <state_interface name="effort"/>
+    </joint>
+    <joint name="joint2">
+      <command_interface name="position">
+        <param name="min">-3.14</param>
+        <param name="max">3.14</param>
+      </command_interface>
+      <state_interface name="position">
+        <param name="initial_value">0.0</param>
+      </state_interface>
+      <state_interface name="velocity"/>
+      <state_interface name="effort"/>
+    </joint>
+    <joint name="joint3">
+      <command_interface name="position">
+        <param name="min">-3.14</param>
+        <param name="max">3.14</param>
+      </command_interface>
+      <state_interface name="position">
+        <param name="initial_value">0.0</param>
+      </state_interface>
+      <state_interface name="velocity"/>
+      <state_interface name="effort"/>
+    </joint>
+    <joint name="joint4">
+      <command_interface name="position">
+        <param name="min">-3.14</param>
+        <param name="max">3.14</param>
+      </command_interface>
+      <state_interface name="position">
+        <param name="initial_value">0.0</param>
+      </state_interface>
+      <state_interface name="velocity"/>
+      <state_interface name="effort"/>
+    </joint>
+    <joint name="joint5">
+      <command_interface name="position">
+        <param name="min">-3.14</param>
+        <param name="max">3.14</param>
+      </command_interface>
+      <state_interface name="position">
+        <param name="initial_value">0.0</param>
+      </state_interface>
+      <state_interface name="velocity"/>
+      <state_interface name="effort"/>
+    </joint>
+    <joint name="joint6">
+      <command_interface name="position">
+        <param name="min">-3.14</param>
+        <param name="max">3.14</param>
+      </command_interface>
+      <state_interface name="position">
+        <param name="initial_value">0.0</param>
+      </state_interface>
+      <state_interface name="velocity"/>
+      <state_interface name="effort"/>
+    </joint>
+  </ros2_control>
     <gazebo>
-      <plugin filename="libgazebo_ros2_control.so" name="gazebo_ros2_control">
-        <robot_param>robot_description</robot_param>
-        <robot_param_node>robot_state_publisher</robot_param_node>
-        <parameters>$(find gazebo_simulation_ros2)/config/fake_ros2_control.yaml</parameters>
-      <!-- <parameters>$(find manta_v2_gazebo_ros2_control)/config/manta_v2_trajectory_controller.yaml</parameters> -->
+    <plugin filename="libgazebo_ros2_control.so" name="gazebo_ros2_control">
+      <parameters>$(find gazebo_simulation_ros2)/config/fake_ros2_control.yaml</parameters>
     </plugin>
   </gazebo>
-  <!-- ros2_control -->
-<ros2_control name="GazeboSystem" type="system">
-  <hardware>
-    <plugin>gazebo_ros2_control/GazeboSystem</plugin>
-    </hardware>
-</ros2_control>
 </robot>

Commit message: modify urdf and xacro

File: urdf/mycobot_280_m5.urdf.xacro (robot description, xacro)
@@ -209,10 +209,15 @@
     <origin xyz= "0 0.0486 -0.007" rpy = "-1.5708 0 0"/>
   </joint>
-<link name="world"/>
+<!-- <link name="world"/>
 <joint name="fixed" type="fixed">
   <parent link="world"/>
   <child link="link1"/>
+</joint> -->
+<link name="base_link"/>
+<joint name="fixed" type="fixed">
+  <parent link="base_link"/>
+  <child link="link1"/>
 </joint>
-  <ros2_control name="GazeboSystem" type="system">
+  <!-- <ros2_control name="GazeboSystem" type="system">
     <hardware>
       <plugin>gazebo_ros2_control/GazeboSystem</plugin>
@@ -289,4 +294,4 @@
       <parameters>$(find gazebo_simulation_ros2)/config/fake_ros2_control.yaml</parameters>
     </plugin>
-  </gazebo>
+  </gazebo> -->
 </robot>
