Commit message: add files for gazebo + moveit2

File: urdf/mycobot_280_m5.urdf.xacro (robot description, xacro)
@@ -209,9 +209,4 @@
     <origin xyz= "0 0.0486 -0.007" rpy = "-1.5708 0 0"/>
   </joint>
-<!-- <link name="world"/>
-<joint name="fixed" type="fixed">
-  <parent link="world"/>
-  <child link="link1"/>
-</joint> -->
 <link name="base_link"/>
 <joint name="fixed" type="fixed">
@@ -219,79 +214,3 @@
   <child link="link1"/>
 </joint>
-  <!-- <ros2_control name="GazeboSystem" type="system">
-    <hardware>
-      <plugin>gazebo_ros2_control/GazeboSystem</plugin>
-    </hardware>
-    <joint name="joint1">
-      <command_interface name="position">
-        <param name="min">-3.15</param>
-        <param name="max">3.14</param>
-      </command_interface>
-      <state_interface name="position">
-        <param name="initial_value">0.0</param>
-      </state_interface>
-      <state_interface name="velocity"/>
-      <state_interface name="effort"/>
-    </joint>
-    <joint name="joint2">
-      <command_interface name="position">
-        <param name="min">-3.14</param>
-        <param name="max">3.14</param>
-      </command_interface>
-      <state_interface name="position">
-        <param name="initial_value">0.0</param>
-      </state_interface>
-      <state_interface name="velocity"/>
-      <state_interface name="effort"/>
-    </joint>
-    <joint name="joint3">
-      <command_interface name="position">
-        <param name="min">-3.14</param>
-        <param name="max">3.14</param>
-      </command_interface>
-      <state_interface name="position">
-        <param name="initial_value">0.0</param>
-      </state_interface>
-      <state_interface name="velocity"/>
-      <state_interface name="effort"/>
-    </joint>
-    <joint name="joint4">
-      <command_interface name="position">
-        <param name="min">-3.14</param>
-        <param name="max">3.14</param>
-      </command_interface>
-      <state_interface name="position">
-        <param name="initial_value">0.0</param>
-      </state_interface>
-      <state_interface name="velocity"/>
-      <state_interface name="effort"/>
-    </joint>
-    <joint name="joint5">
-      <command_interface name="position">
-        <param name="min">-3.14</param>
-        <param name="max">3.14</param>
-      </command_interface>
-      <state_interface name="position">
-        <param name="initial_value">0.0</param>
-      </state_interface>
-      <state_interface name="velocity"/>
-      <state_interface name="effort"/>
-    </joint>
-    <joint name="joint6">
-      <command_interface name="position">
-        <param name="min">-3.14</param>
-        <param name="max">3.14</param>
-      </command_interface>
-      <state_interface name="position">
-        <param name="initial_value">0.0</param>
-      </state_interface>
-      <state_interface name="velocity"/>
-      <state_interface name="effort"/>
-    </joint>
-  </ros2_control>
-    <gazebo>
-    <plugin filename="libgazebo_ros2_control.so" name="gazebo_ros2_control">
-      <parameters>$(find gazebo_simulation_ros2)/config/fake_ros2_control.yaml</parameters>
-    </plugin>
-  </gazebo> -->
 </robot>

File: urdf/mycobot_280_m5_gazebo_config.xacro (robot description, xacro)
@@ -1,4 +1,5 @@
 <?xml version="1.0"?>
 <robot  xmlns:xacro="http://www.ros.org/wiki/xacro" name="mycobot_ai_no" >
+  <!-- <xacro:include filename="$(find gazebo_simulation_ros2)/urdf/mycobot.trans" /> -->
   <xacro:include filename="$(find gazebo_simulation_ros2)/urdf/mycobot_280_m5.urdf.xacro" />
   <ros2_control name="GazeboSystem" type="system">
@@ -8,5 +9,5 @@
     <joint name="joint1">
       <command_interface name="position">
-        <param name="min">-3.15</param>
+        <param name="min">-3.14</param>
         <param name="max">3.14</param>
       </command_interface>
@@ -75,5 +76,7 @@
     <gazebo>
     <plugin filename="libgazebo_ros2_control.so" name="gazebo_ros2_control">
-      <parameters>$(find gazebo_simulation_ros2)/config/fake_ros2_control.yaml</parameters>
+      <robot_param>robot_description</robot_param>
+      <robot_param_node>robot_state_publisher</robot_param_node>
+      <parameters>$(find gazebo_simulation_ros2)/config/mycobot_move_group_controller.yaml</parameters>
     </plugin>
   </gazebo>

Commit message: update urdf

File: urdf/mycobot_280_m5.urdf.xacro (robot description, xacro)
@@ -209,6 +209,11 @@
     <origin xyz= "0 0.0486 -0.007" rpy = "-1.5708 0 0"/>
   </joint>
+<link name="world"/>
 <link name="base_link"/>
-<joint name="fixed" type="fixed">
+<joint name="world_joint" type="fixed">
+  <parent link="world"/>
+  <child link="base_link"/>
+</joint>
+<joint name="base_joint" type="fixed">
   <parent link="base_link"/>
   <child link="link1"/>
